Commit message: a

File: src/hardware/urdf/arm.urdf (robot description, URDF)
Before this commit: robot arm, 7 links, 6 joints
Links:
- link base: geometry collision mesh filename=package://hardware/urdf/assets/base.stl; collision mesh filename=package://hardware/urdf/assets/mg995.stl
- link part_14: geometry collision mesh filename=package://hardware/urdf/assets/part_14.stl; collision mesh filename=package://hardware/urdf/assets/simplified_claw_attachment.s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
- link part_15: geometry collision mesh filename=package://hardware/urdf/assets/mg995.stl; collision mesh filename=package://hardware/urdf/assets/part_15.stl
- link part_7: geometry collision mesh filename=package://hardware/urdf/assets/part_7.stl; visual mesh filename=package://hardware/urdf/assets/part_7.stl
- link part_8: geometry collision mesh filename=package://hardware/urdf/assets/mg995.stl; collision mesh filename=package://hardware/urdf/assets/part_8.stl
- link part_9: geometry collision mesh filename=package://hardware/urdf/assets/part_9.stl; collision mesh filename=package://hardware/urdf/assets/sg90_v1.stl

File: src/hardware/urdf/arm.urdf.xacro (robot description, xacro)
@@ -1,5 +1,5 @@
 <?xml version="1.0"?>
 <robot xmlns:xacro="http://www.ros.org/wiki/xacro" name="arm">
-  <xacro:include filename="$(find arm)/urdf/arm.urdf" />
+  <xacro:include filename="$(find hardware)/urdf/arm.urdf" />
   <!-- ros2_control configuration -->
   <ros2_control name="arm" type="system">
