Commit message: moved urdf to its own package

File: src/moveit2/config/arm.urdf.xacro (robot description, xacro)
@@ -3,5 +3,5 @@
     <xacro:arg name="initial_positions_file" default="initial_positions.yaml" />
     <!-- Import arm urdf file -->
-    <xacro:include filename="$(find hardware)/urdf/arm.urdf" />
+    <xacro:include filename="$(find robot_description)/urdf/arm.urdf" />
     <!-- Import control_xacro -->
     <xacro:include filename="arm.ros2_control.xacro" />

File: src/robot_description/urdf/arm.urdf (robot description, URDF)
Before this commit: robot arm, 7 links, 6 joints
Links:
- link base: geometry collision mesh filename=package://robot_description/urdf/assets/base.stl; collision mesh filename=package://robot_description/urdf/assets/mg995.stl
- link part_14: geometry collision mesh filename=package://robot_description/urdf/assets/part_14.stl; collision mesh filename=package://robot_description/urdf/assets/simplified_claw_att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
- link part_15: geometry collision mesh filename=package://robot_description/urdf/assets/mg995.stl; collision mesh filename=package://robot_description/urdf/assets/part_15.stl
- link part_7: geometry collision mesh filename=package://robot_description/urdf/assets/part_7.stl; visual mesh filename=package://robot_description/urdf/assets/part_7.stl
- link part_8: geometry collision mesh filename=package://robot_description/urdf/assets/mg995.stl; collision mesh filename=package://robot_description/urdf/assets/part_8.stl
- link part_9: geometry collision mesh filename=package://robot_description/urdf/assets/part_9.stl; collision mesh filename=package://robot_description/urdf/assets/sg90_v1.stl

File: src/robot_description/urdf/arm.urdf.xacro (robot description, xacro)
@@ -1,5 +1,5 @@
 <?xml version="1.0"?>
 <robot xmlns:xacro="http://www.ros.org/wiki/xacro" name="arm">
-  <xacro:include filename="$(find hardware)/urdf/arm.urdf" />
+  <xacro:include filename="$(find robot_description)/urdf/arm.urdf" />
   <!-- ros2_control configuration -->
   <ros2_control name="arm" type="system">
